Commit message: cg changed

File: urdf/rosarm.urdf.xacro (robot description, xacro)
@@ -21,5 +21,5 @@
 		<collision name="collision_base">
 			<geometry>
-				<box size="0.2 0.2 0.07"/>
+					<box size="${l1} ${b1} ${h1}"/>
 			</geometry>
 		</collision>
@@ -73,5 +73,5 @@
 		</visual>
 		<collision name="collision_link_1">
-			<origin rpy="0 0 0" xyz="0 0 0"/>
+			<origin rpy="0 0 0" xyz="0 0 ${l3/2}"/>
 			<geometry>
 				<cylinder length="${l3}" radius="${r3}"/>
@@ -80,5 +80,5 @@
 		<inertial>
 			<mass value="${m3}"/>
-			<origin rpy="0 0 0" xyz="0 0 0"/>
+			<origin rpy="0 0 0" xyz="0 0 ${l3/2}"/>
 			<inertia ixx="${m3*((3*r3*r3)+(l3*l3))/12.0}" ixy="0" ixz="0" iyy="${m3*((3*r3*r3)+(l3*l3))/12.0}" iyz="0" izz="${(m3*r3*r3)/2.0}"/>
 		</inertial>
@@ -101,5 +101,5 @@
 		</visual>
 		<collision name="collision_link_1">
-			<origin rpy="0 0 0" xyz="0 0 0"/>
+			<origin rpy="0 0 0" xyz="0 0 ${l3/2}"/>
 			<geometry>
 				<cylinder length="${l3}" radius="${r3}"/>
@@ -108,5 +108,5 @@
 		<inertial>
 			<mass value="${m3}"/>
-			<origin rpy="0 0 0" xyz="0 0 0"/>
+			<origin rpy="0 0 0" xyz="0 0 ${l3/2}"/>
 			<inertia ixx="${m3*((3*r3*r3)+(l3*l3))/12.0}" ixy="0" ixz="0" iyy="${m3*((3*r3*r3)+(l3*l3))/12.0}" iyz="0" izz="${(m3*r3*r3)/2.0}"/>
 		</inertial>
@@ -129,5 +129,5 @@
 		</visual>
 		<collision name="collision_link_1">
-			<origin rpy="0 0 0" xyz="0 0 0"/>
+			<origin rpy="0 0 0" xyz="0 0 ${l3/2}"/>
 			<geometry>
 				<cylinder length="${l3}" radius="${r3}"/>
@@ -136,5 +136,5 @@
 		<inertial>
 			<mass value="${m3}"/>
-			<origin rpy="0 0 0" xyz="0 0 0"/>
+			<origin rpy="0 0 0" xyz="0 0 ${l3/2}"/>
 			<inertia ixx="${m3*((3*r3*r3)+(l3*l3))/12.0}" ixy="0" ixz="0" iyy="${m3*((3*r3*r3)+(l3*l3))/12.0}" iyz="0" izz="${(m3*r3*r3)/2.0}"/>
 		</inertial>
@@ -144,5 +144,5 @@
 		<child link="link_3"/>
 		<parent link="link_2"/>
-		<axis xyz="1 1 0"/>
+		<axis xyz="1 0 0"/>
 		<limit upper="3.14" lower="-3.14" effort="10000" velocity="1000"/>
 		<joint_properties damping="1.0" friction="1.0"/>

Commit message: Update

File: urdf/rosarm.urdf.xacro (robot description, xacro)
@@ -88,5 +88,5 @@
 		<child link="link_1"/>
 		<parent link="base_z"/>
-		<axis xyz="1 1 0"/>
+		<axis xyz="1 0 0"/>
 		<limit upper="3.14" lower="-3.14" effort="10000" velocity="1000"/>
 		<joint_properties damping="1.0" friction="1.0"/>
@@ -148,5 +148,5 @@
 		<joint_properties damping="1.0" friction="1.0"/>
 	</joint>
- <xacro:include filename="$(find rosarm_pkg)/urdf/rosarm_transmission.urdf" />
+ <xacro:include filename="$(find rosarm_pkg)/urdf/rosarm_transmission1.urdf" />
  <xacro:include filename="$(find rosarm_pkg)/urdf/rosarm_plugin.urdf" />
 </robot>

Commit message: Surroundings added

File: urdf/rosarm.urdf.xacro (robot description, xacro)
@@ -7,8 +7,10 @@
 	 <color rgba="1 1 1 1"/>
  </material>
+	<link name="world"/>
  <xacro:property name="m" value="2" />
  <xacro:property name="l1" value="0.15" />
  <xacro:property name="b1" value="0.15" />
  <xacro:property name="h1" value="0.15" />
+ <xacro:include filename="$(find rosarm_pkg)/urdf/surroundings.urdf" />
 	<link name="base_link">
 		<visual>
@@ -30,4 +32,9 @@
 		</inertial>
 	</link>
+	<joint name="world_to_base" type="fixed">
+		<parent link="world"/>
+		<child link="base_link"/>
+		<origin xyz="0 0 ${ht+h1/2}" rpy="0 0 0"/>
+	</joint>
  <xacro:property name="l2" value="0.08" />
  <xacro:property name="r2" value="0.075" />

Commit message: Update

File: urdf/rosarm.urdf.xacro (robot description, xacro)
@@ -35,5 +35,5 @@
 		<parent link="world"/>
 		<child link="base_link"/>
-		<origin xyz="0 0 ${ht+h1/2}" rpy="0 0 0"/>
+		<origin xyz="0 0.5 ${ht+h1/2}" rpy="0 0 0"/>
 	</joint>
  <xacro:property name="l2" value="0.08" />

Commit message: Update

File: urdf/rosarm.urdf.xacro (robot description, xacro)
@@ -1,4 +1,4 @@
 <?xml version="1.0"?>
-<robot name="rosarm" xmlns:xacro="http://www.ros.org/wiki/xacro" >
+<robot name="rosarm" xmlns:xacro="http://ros.org/wiki/xacro" >
  <material name="blue">
  	<color rgba="0 0 0.8 1"/>
@@ -12,5 +12,4 @@
  <xacro:property name="b1" value="0.15" />
  <xacro:property name="h1" value="0.15" />
- <xacro:include filename="$(find rosarm_pkg)/urdf/surroundings.urdf.xacro" />
 	<link name="base_link">
 		<visual>
@@ -35,5 +34,5 @@
 		<parent link="world"/>
 		<child link="base_link"/>
-		<origin xyz="0 0.5 ${ht+h1/2}" rpy="0 0 0"/>
+		<origin xyz="0 0.5 ${h1/2}" rpy="0 0 0"/>
 	</joint>
  <xacro:property name="l2" value="0.08" />

File: urdf/surroundings.urdf.xacro (robot description, xacro)
@@ -1,4 +1,4 @@
 <?xml version="1.0" ?>
-<robot name="rosarm" xmlns:xacro="http://ros.org/wiki/xacro">
+<robot name="surroundings" xmlns:xacro="http://ros.org/wiki/xacro">
  <xacro:property name="mt" value="2" />
  <xacro:property name="lt" value="1" />
@@ -31,33 +31,3 @@
 		<origin xyz="0 0 ${ht/2}" rpy="0 0 0"/>
 	</joint>
- <xacro:property name="mk" value="0.2" />
- <xacro:property name="lk" value="0.3" />
- <xacro:property name="bk" value="0.1" />
- <xacro:property name="hk" value="0.05" />
-	<link name="kinect">
-		<visual>
-			<origin rpy="0 0 0" xyz="0 0 0"/>
-			<geometry>
-					<box size="${lk} ${bk} ${hk}"/>
-			</geometry>
-		</visual>
-		<collision name="collision_kinect">
-			<geometry>
-					<box size="${lt} ${bt} ${ht}"/>
-			</geometry>
-		</collision>
-		<inertial>
-			<mass value="${mk}"/>
-			<origin rpy="0 0 0" xyz="0 0 0"/>
-			<inertia ixx="${mk*hk*bk/12.0}" ixy="0" ixz="0" iyy="${mk*lk*hk/12.0}" iyz="0" izz="${mk*lk*bk/12.0}"/>
-		</inertial>
-	</link>
-	<gazebo reference="kinect">
-  		<material>Gazebo/Black</material>
-	</gazebo>
-	<joint name="world_to_kinect" type="fixed">
-		<parent link="world"/>
-		<child link="kinect"/>
-		<origin xyz="0 -1 1" rpy="0 0 0"/>
-	</joint>
-</robot>
+ </robot>
