Commit message: Bug Solved

File: urdf/kinect.urdf.xacro (robot description, xacro)
@@ -7,5 +7,5 @@
 	<link name="kinect">
 		<visual>
-			<origin rpy="0 0 0" xyz="0 0 0"/>
+			<origin rpy="0 0 1.5707" xyz="0 0 0"/>
 			<geometry>
 					<box size="${lk} ${bk} ${hk}"/>
@@ -29,5 +29,11 @@
 		<parent link="world"/>
 		<child link="kinect"/>
-		<origin xyz="0 0 0.5" rpy="0 0 1.5707"/>
+		<origin xyz="0 0 0.5" rpy="0 0 0"/>
+	</joint>
+	<link name="kinect_link" />
+	<joint name="kinect_joint" type="fixed">
+		<parent link="kinect"/>
+		<child link="kinect_link"/>
+		<origin xyz="0 0 0" rpy="-1.5707 0 0"/>
 	</joint>
 	  <!-- camera -->
@@ -54,5 +60,5 @@
 		        <updateRate>10.0</updateRate>
 		        <cameraName>kinect</cameraName>
-		        <frameName>kinect</frameName>
+		        <frameName>kinect_link</frameName>
 		    <imageTopicName>rgb/image_raw</imageTopicName>
 		    <depthImageTopicName>depth/image_raw</depthImageTopicName>

Commit message: Kinect placement

File: urdf/kinect.urdf.xacro (robot description, xacro)
@@ -3,9 +3,9 @@
  <xacro:property name="mk" value="0.1" />
  <xacro:property name="lk" value="0.05" />
- <xacro:property name="bk" value="0.2" />
- <xacro:property name="hk" value="0.05" />
+ <xacro:property name="bk" value="0.05" />
+ <xacro:property name="hk" value="0.2" />
 	<link name="kinect">
 		<visual>
-			<origin rpy="0 0 1.5707" xyz="0 0 0"/>
+			<origin rpy="0 0 0" xyz="0 0 0"/>
 			<geometry>
 					<box size="${lk} ${bk} ${hk}"/>
@@ -29,5 +29,5 @@
 		<parent link="world"/>
 		<child link="kinect"/>
-		<origin xyz="0 0 0.5" rpy="0 0 0"/>
+		<origin xyz="0 -0.01 2" rpy="0 1.5707 0"/>
 	</joint>
 	<link name="kinect_link" />
@@ -35,5 +35,5 @@
 		<parent link="kinect"/>
 		<child link="kinect_link"/>
-		<origin xyz="0 0 0" rpy="-1.5707 0 0"/>
+		<origin xyz="0 0 0" rpy="0 0 0"/>
 	</joint>
 	  <!-- camera -->

File: urdf/rosarm.urdf.xacro (robot description, xacro)
@@ -9,4 +9,5 @@
 	<link name="world"/>
  <xacro:include filename="$(find rosarm_pkg)/urdf/kinect.urdf.xacro" />
+ <xacro:include filename="$(find rosarm_pkg)/urdf/table.urdf.xacro" />
  <xacro:property name="m" value="2" />
  <xacro:property name="l1" value="0.15" />
@@ -35,5 +36,5 @@
 		<parent link="world"/>
 		<child link="base_link"/>
-		<origin xyz="0 0.5 ${h1/2}" rpy="0 0 0"/>
+		<origin xyz="0 0.3 ${ht+h1/2}" rpy="0 0 0"/>
 	</joint>
  <xacro:property name="l2" value="0.08" />

File: urdf/table.urdf.xacro (robot description, xacro)
@@ -1,4 +1,4 @@
 <?xml version="1.0" ?>
-<robot name="surroundings" xmlns:xacro="http://ros.org/wiki/xacro">
+<robot name="table" xmlns:xacro="http://ros.org/wiki/xacro">
  <xacro:property name="mt" value="2" />
  <xacro:property name="lt" value="1" />

Commit message: Update

File: urdf/kinect.urdf.xacro (robot description, xacro)
@@ -29,5 +29,5 @@
 		<parent link="world"/>
 		<child link="kinect"/>
-		<origin xyz="0 -0.01 2" rpy="0 1.5707 0"/>
+		<origin xyz="0 -0.01 2.5" rpy="0 1.5707 0"/>
 	</joint>
 	<link name="kinect_link" />
